File: redox/pcb/rev1.0/hotswap-left/redox_rev1.kicad_sch (KiCad schematic)
At the start: 75 parts, among them K0 KEYSW, K1 KEYSW, K10 KEYSW, K11 KEYSW, K12 KEYSW, K13 KEYSW, K14 KEYSW, K15 KEYSW, K16 KEYSW, K2 KEYSW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

Commit message: Complete left PCB
Parts:
- D0, D1, D10, D11, D12, D13, D14, D15, D16, D2, D20, D21, D22, D23, D24, D25, D26, D3, D30, D31, D32, D33, D34, D35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: footprint redox_footprints:Diode-dual -> redox_footprints:Diode-smd-via
