File: redox/pcb/rev1.0/hotswap-right/redox_rev1.kicad_pcb (KiCad board)
At the start: 2 copper layers, 162.2 x 126.5 mm, 82 parts, among them K0 KEYSW, K1 KEYSW, K10 KEYSW, K11 KEYSW, K12 KEYSW, K13 KEYSW, K14 KEYSW, K15 KEYSW, K16 KEYSW, K2 KEYSW, K20 KEYSW, K21 KEYSW, K22 KEYSW, K23 KEYSW, K24 KEYSW, K25 KEYSW, K26 KEYSW, K3 KEYSW, K30 KEYSW, K31 KEYSW, K32 KEYSW, K33 KEYSW, K34 KEYSW, K35 KEYSW, K36 KEYSW, K4 KEYSW, K40 KEYSW, K41 KEYSW, K42 KEYSW, K43 KEYSW, K44 KEYSW, K45 KEYSW, K46 KEYSW, K5 KEYSW, K6 KEYSW, U1 ProMicro

Commit message: Complete right PCB
Parts:
- removed R1, R2: 4.7k, redox_footprints:Resistor-Compact
Routing:
- net col5: track 57.2 -> 186.7 mm, vias 0 -> 1
- net row0: track 0.00 -> 128.7 mm
- net col6: track 124.4 -> 225.0 mm, vias 0 -> 2
- net VCC: track 0.00 -> 87.2 mm
- net SCL: track 0.00 -> 70.0 mm
- net col3: track 38.1 -> 104.3 mm
- net row4: track 127.1 -> 190.5 mm, vias 0 -> 1
- net col4: track 84.9 -> 143.6 mm, vias 0 -> 1
- net SDA: track 0.00 -> 58.3 mm
- net col0: track 77.3 -> 129.3 mm
- net row3: track 133.8 -> 183.5 mm, vias 0 -> 1
- net row2: track 121.5 -> 155.6 mm, vias 0 -> 1
- net RST: track 0.00 -> 31.1 mm
- net Net-(D45-Pad2): track 0.00 -> 25.5 mm
- net col1: track 76.2 -> 100.4 mm
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